File: ActiveSpiceExampleSCH/01_ActiveSpice_LogicGate_AOPideal_000.kicad_sch (KiCad schematic)
At the start: 49 parts, among them U1 Inverter, U10 Inverter, U11 Inverter, U12 ${SIM.PARAMS}, U13 ${SIM.PARAMS}, U14 ${SIM.PARAMS}, U15 ${SIM.PARAMS}, U16 Spice-Switch, U17 Spice_BeaviorFct, U2 AND, U3 NAND, U4 OR, U5 NOR, U6 XOR, U7 NAND, U8 NAND, U9 XNOR

Commit message: update lib Activespice and shape it
Parts:
- removed U: XNOR, symbol 74xx:74LS86
- removed U (x3), U14: ${SIM.PARAMS}, symbol Simulation_SPICE:OPAMP
- removed U: XOR, symbol 74xx:74LS86
- removed U: OR, symbol 74xx:74LS86
- removed U: NOR, symbol 74xx:74LS86
- removed U, U10, U11: Inverter, symbol 74xx:74LS86
- removed U: AND, symbol 74xGxx:74AUC2G08
- removed U, U7, U8: NAND, symbol 74xGxx:74AUC2G08
- removed U1: Inverter, symbol 0x190FULL_SpiceOnly:INVERTER
- removed U12: ${SIM.PARAMS}, symbol 0x190FULL_SpiceOnly:OPAMP_ideal_V+top
- removed U13: ${SIM.PARAMS}, symbol 0x190FULL_SpiceOnly:OPAMP_ideal_V-top
- removed U15: ${SIM.PARAMS}, symbol 0x190FULL_SpiceOnly:RECTIFIER
- removed U16: Spice-Switch, symbol 0x190FULL_SpiceOnly:Spice-Switch-1x2-ideal_alterable
- removed U17: Spice_BeaviorFct, symbol 0x190FULL_SpiceOnly:Behavioral_Fonction_alterable
- removed U2: AND, symbol 0x190FULL_SpiceOnly:AND
- removed U3: NAND, symbol 0x190FULL_SpiceOnly:NAND
- removed U4: OR, symbol 0x190FULL_SpiceOnly:OR
- removed U5: NOR, symbol 0x190FULL_SpiceOnly:NOR
- removed U6: XOR, symbol 0x190FULL_SpiceOnly:XOR
- removed U9: XNOR, symbol 0x190FULL_SpiceOnly:XNOR
- added U1, U6, U8: Inverter, symbol 0xActiveSpice:INVERTER
- added U10: Schmitt-trigger, symbol 74xGxx:74LVC1GU04DRL
- added U15: XOR, symbol 0xActiveSpice:LogicGate_XOR
- added U16: ${SIM.PARAMS}, symbol 0xActiveSpice:OPAMP_ideal_V+top
- added U17: XNOR, symbol 0xActiveSpice:LogicGate_XNOR
- added U19: Spice-Switch, symbol 0xActiveSpice:Spice-Switch-1x2-ideal_alterable
- added U2: RSFlipFlop, symbol 0xActiveSpice:FlipFlop_RS
- added U20, U4: ${SIM.PARAMS}, symbol 0xActiveSpice:OPAMP_ideal_V-top
- added U21: OR, symbol 0xActiveSpice:LogicGate_OR
- added U22: NOR, symbol 0xActiveSpice:LogicGate_NOR
- added U23, U3, U5: NAND, symbol 0xActiveSpice:LogicGate_NAND
- added U24: AND, symbol 0xActiveSpice:LogicGate_AND
- added U7: ${SIM.PARAMS}, symbol 0xActiveSpice:Fct_Rectifier_Full
- added U9: Spice_BeaviorFct, symbol 0xActiveSpice:Behavioral_Fonction_alterable
- added V3, V5, V9: VPULSE, symbol Simulation_SPICE:VPULSE
- C1: renamed from C2; value 10p -> 10f
- C2: renamed from C1; value 30p -> 30f
- C3, C4: value 100n -> 10n
- R10, R9: value 8K -> 1K
- R11: value 6K -> 1K
- R12: value 10K -> 1K
- R3: renamed from R1; value 10K -> 1K
- R4: renamed from R2; value 10K -> 1K
- V7: renamed from V4; value 0.5 -> 1
- renumbered R3 to R1, R4 to R2, V9 to V1, V1 to V2, V2 to V4, V3 to V6, V5 to V8
Connections:
- net 0: now also U1.2 (G), U10.2 (G), U15.2 (G), U17.2 (G), U2.2 (G), U20.3 (P), U21.2 (G), U22.2 (G), U23.2 (G), U24.2 (G), U3.2 (G), U5.2 (G), U6.2 (G), U8.2 (G), U9.4 (GND), V3.2, V5.2, V9.2
- net AND_S: now also U24.5 (S)
- net Inv: now also U1.4 (S)
- net NAND_S: now also U23.5 (S)
- net NOR_S: now also U22.5 (S)
- net OR_S: now also U21.5 (S)
- net QFlipflop: now also U5.5 (S)
- net RSFlipFlop: now also U3.5 (S)
- net Res: now also U15.4 (B), U17.4 (B), U19.1, U21.4 (B), U22.4 (B), U23.4 (B), U24.4 (B), U8.3 (A), U9.2 (B)
- net Set: now also U1.3 (A), U15.3 (A), U17.3 (A), U19.2, U21.3 (A), U22.3 (A), U23.3 (A), U24.3 (A), U6.3 (A), U9.1 (A)
- net VCCQ: now also U1.1 (VCC), U10.1 (VCC), U15.1 (VCC), U16.1 (VCC), U17.1 (VCC), U2.1 (VCC), U20.1 (VCC), U21.1 (VCC), U22.1 (VCC), U23.1 (VCC), U24.1 (VCC), U3.1 (VCC), U4.1 (VCC), U5.1 (VCC), U6.1 (VCC), U8.1 (VCC)
- net VSS: now also U16.2 (G), U20.2 (G), U4.2 (G)
- net Vin: now also U16.3 (P), U7.1 (I)
- net XNOR_S: now also U17.5 (S)
- net XOR_S: now also U15.5 (S)
- net gs: now also U20.5 (S)
- net gs2: now also U16.5 (S)
- net gs3: now also U4.5 (S)
- net rec: now also U7.2 (S)
- net at R7.2, R8.1: now also U16.4 (M)
- net at R11.2, R12.1: now also U4.4 (M)
- net at R5.2, R6.1: now also U20.4 (M)
- net at C4.2, R10.2: now also U4.3 (P)
- net at C1.1, R1.2: now also U3.4 (B)
- net at C2.1, R2.2: now also U5.3 (A)
- new net: U10.3 (In), V9.1
- new net: U5.4 (B), U8.4 (S)
- new net: U3.3 (A), U6.4 (S)
- new net Math: U9.3 (X)
- new net OutRS: U2.5 (Q)
- new net OutTrigged: U10.4 (Q)
- new net Q: U2.6 (~{Q})
- new net Sw1: U19.3
- new net Sw2: U19.4
- new net res2: U2.4 (Res), V5.1
- new net set2: U2.3 (Set), V3.1
Other:
- note added: ".tran 1n 25u 0 uic *.options cshunt = 1e-13 *.OPTIONS ITL1=2000 *.OPTIONS RELTOL=.01 *.control *run *gnuplot time V(Set) V(Res) V(AND_S) *gnuplot multiplot *set origin 0.0,0.5 *gnuplot V(Set) time V(Res) V(AND_S) *set origin 0.0,0.0 *plot time V(Set) V(Res) V(OR_S) *unset multiplot *plot V(select) V(OutA) V(OutB) *.endc"
- note added: "color : #9592C2BF"
- note added: "reference to ground... may 10T to 0 loop determination by delay"
- note removed: ".tran 10n 250u 0 uic *.options cshunt = 1e-13 *.OPTIONS ITL1=2000 *.OPTIONS RELTOL=.01 *.control *run *gnuplot time V(Set) V(Res) V(AND_S) *gnuplot multiplot *set origin 0.0,0.5 *gnuplot V(Set) time V(Res) V(AND_S) *set origin 0.0,0.0 *plot time V(Set) V(Res) V(OR_S) *unset multiplot *plot V(select) V(OutA) V(OutB) *.endc"
